File: projects/Serial_NTP_clock/PCB_board_clock.brd (EAGLE design)
At the start: 130 x 60 mm, 37 parts, among them IC1 74HC595N, IC2 7805T, IC3 LD117AV, J1 DCJ0202

Commit message: Grounded plate, relocated module of scheme and added more vias
Connections:
- new net N$11: U$1.D12
- net DATA_PIN: no longer U$1.D12
Routing:
- net N$9: track 19.4 -> 0.00 mm
- added copper zone on layer 1, net GND
Changed lines of the file:
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@@
 <wire x1="45.72" y1="7.62" x2="39.37" y2="7.62" width="0.5" layer="16"/>
 <wire x1="39.37" y1="7.62" x2="36.83" y2="5.08" width="0.5" layer="16"/>
+<polygon width="0.1016" layer="1" isolate="0.4064" orphans="yes">
+<vertex x="8.7" y="76.5"/>
+<vertex x="-24.9" y="42.9"/>
+<vertex x="-24.9" y="4.8"/>
+<vertex x="-5.1" y="-15"/>
+<vertex x="155.4" y="-15"/>
+<vertex x="155.4" y="73.2"/>
+<vertex x="146.4" y="82.2"/>
+<vertex x="14.4" y="82.2"/>
+</polygon>
 </signal>
 <signal name="VCC">
@@
 </signal>
 <signal name="DATA_PIN">
-<contactref element="U$1" pad="D12"/>
 <contactref element="IC1" pad="14"/>
-<wire x1="16.97273125" y1="5.08" x2="16.51" y2="5.08" width="0.4" layer="16"/>
 <wire x1="18.63313125" y1="3.4196" x2="16.97273125" y2="5.08" width="0.4" layer="16"/>
 <wire x1="48.26" y1="7.62" x2="44.0596" y2="3.4196" width="0.4" layer="16"/>
@@
 <wire x1="45.3086" y1="42.42420625" x2="50.58439375" y2="47.7" width="0.4" layer="16"/>
 <wire x1="50.58439375" y1="47.7" x2="67.05728125" y2="47.7" width="0.4" layer="16"/>
-</signal>
-<signal name="N$31">
-<contactref element="R4" pad="1"/>
-<contactref element="U$1" pad="D7"/>
-<wire x1="16.51" y1="20.32" x2="19.19" y2="23" width="0.4" layer="1"/>
-<wire x1="29.8387875" y1="23" x2="30.2511875" y2="23.4124" width="0.4" layer="1"/>
-<wire x1="33.5724" y1="23.4124" x2="34.29" y2="24.13" width="0.4" layer="1"/>
-<wire x1="30.2511875" y1="23.4124" x2="33.5724" y2="23.4124" width="0.4" layer="1"/>
-<wire x1="19.19" y1="23" x2="29.8387875" y2="23" width="0.4" layer="1"/>
 </signal>
 <signal name="N$32">
@@
 <wire x1="69.85" y1="5.08" x2="66.04" y2="5.08" width="0.5" layer="1"/>
 </signal>
+<signal name="N$9">
+<contactref element="R4" pad="1"/>
+<contactref element="U$1" pad="D7"/>
+<wire x1="16.51" y1="20.32" x2="34.29" y2="24.13" width="0" layer="19" extent="1-1"/>
+</signal>
+<signal name="N$11">
+<contactref element="U$1" pad="D12"/>
+</signal>
 </signals>
